File: Breadboar Power Supply v1/Breadboar Power Supply v1.kicad_pcb (KiCad board)
At the start: 2 copper layers, 30.1 x 52.1 mm, 15 parts, among them J1 Barrel_Jack_Switch, J2 Conn_02x02_Odd_Even, J3 Conn_02x02_Odd_Even, SW1 SW_DPDT_x2, U1 LM7805_TO220

Commit message: filled zones
Routing:
- added copper zone on B.Cu, net /GND
- added copper zone on F.Cu, net /GND
Changed lines of the file:
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@@
   (segment (start 193.489 112.454) (end 192.102 112.454) (width 0.3) (layer F.Cu) (net 9))
   (segment (start 194.31 111.633) (end 193.489 112.454) (width 0.3) (layer F.Cu) (net 9))
+  (zone (net 2) (net_name /GND) (layer F.Cu) (hatch edge 0.508)
+    (connect_pads (clearance 0.508))
+    (min_thickness 0.254)
+    (fill yes (arc_segments 32) (thermal_gap 0.508) (thermal_bridge_width 0.508))
+    (polygon
+      (pts
+        (xy 201.803 90.551) (xy 195.58 90.551) (xy 195.58 129.159) (xy 201.93 129.159) (xy 201.93 135.89)
+        (xy 172.085 135.89) (xy 172.085 84.201) (xy 201.803 84.201)
+      )
+    )
+  )
+  (zone (net 2) (net_name /GND) (layer B.Cu) (hatch edge 0.508)
+    (connect_pads (clearance 0.508))
+    (min_thickness 0.254)
+    (fill yes (arc_segments 32) (thermal_gap 0.508) (thermal_bridge_width 0.508))
+    (polygon
+      (pts
+        (xy 201.803 90.551) (xy 195.58 90.551) (xy 195.58 129.159) (xy 201.93 129.159) (xy 201.93 135.89)
+        (xy 172.085 135.89) (xy 172.085 84.201) (xy 201.803 84.201)
+      )
+    )
+  )
 )

Commit message: Finish layout
Parts:
- added REF**: KiCad-Logo2_5mm_SilkScreen, Symbol:KiCad-Logo2_5mm_SilkScreen, B.Cu at (179.8, 95.6)
- added REF**: OSHW-Logo2_7.3x6mm_SilkScreen, Symbol:OSHW-Logo2_7.3x6mm_SilkScreen, B.Cu at (179.6, 109.5)
- moved R1 0.89 mm to (191.5, 134.0)
Other:
- board text added: "330"
- board text added: "5V"
- board text added: "Breadboard Power Supply v1.0"
- board text added: "GND"
