File: Breadboar Power Supply v1/Breadboar Power Supply v1.kicad_pcb (KiCad board)
At the start: 2 copper layers, 30.1 x 52.1 mm, 17 parts, among them J1 Barrel_Jack_Switch, J2 Conn_02x02_Odd_Even, J3 Conn_02x02_Odd_Even, SW1 SW_DPDT_x2, U1 LM7805_TO220

Commit message: Final PCB
Parts:
- D5, D6: footprint LED_THT:LED_D5.0mm -> LED_SMD:LED_0805_2012Metric
- moved D6 2.43 mm to (192.2, 101.7)
- moved D5 1.92 mm to (192.2, 119.1)
Routing:
- net /GND: track 93.6 -> 96.9 mm, vias 0 -> 2
- net Net-(D5-Pad2): track 16.1 -> 17.6 mm
- net Net-(D6-Pad2): track 11.5 -> 12.8 mm, vias 0 -> 1
Other:
- outline, holes or cut-outs redrawn
