File: Breadboar Power Supply v1/Breadboar Power Supply v1.kicad_pcb (KiCad board)
At the start: 2 copper layers, 30.1 x 52.1 mm, 17 parts, among them J1 Barrel_Jack_Switch, J2 Conn_02x02_Odd_Even, J3 Conn_02x02_Odd_Even, SW1 SW_DPDT_x2, U1 LM7805_TO220

Commit message: my name xd
Other:
- board text added: "Author: Diego Gonzales"

Commit message: extrasssss
Parts:
- removed the REF** at (179.8, 95.6)
- added G***: LOGO, logos:Catcuber_10.9x10.9mm, B.Cu at (179.6, 95.5)
