File: Breadboar Power Supply v1/Breadboar Power Supply v1.sch (KiCad schematic (older format))
At the start: 15 parts, among them J1 Barrel_Jack_Switch, J2 Conn_02x02_Odd_Even, J3 Conn_02x02_Odd_Even, SW1 SW_DPDT_x2, U1 LM7805_TO220

Commit message: Footprints
Parts:
- C1: footprint (none) -> Capacitor_THT:CP_Radial_D10.0mm_P5.00mm
- C2: footprint (none) -> Capacitor_THT:CP_Radial_D6.3mm_P2.50mm
- D5, D6: footprint (none) -> LED_THT:LED_D5.0mm
- J1: footprint (none) -> Connector_BarrelJack:BarrelJack_CUI_PJ-102AH_Horizontal
- J2, J3: footprint (none) -> Connector_PinHeader_2.54mm:PinHeader_2x02_P2.54mm_Vertical
- R1, R2: footprint (none) -> Resistor_THT:R_Axial_DIN0207_L6.3mm_D2.5mm_P7.62mm_Horizontal
- SW1: footprint (none) -> digikey-footprints:Switch_Slide_11.6x4mm_EG1218
Changed lines of the file:
@@
 F 0 "C2" H 5565 3896 50  0000 L CNN
 F 1 "47uF" H 5565 3805 50  0000 L CNN
-F 2 "" H 5450 3850 50  0001 C CNN
+F 2 "Capacitor_THT:CP_Radial_D6.3mm_P2.50mm" H 5450 3850 50  0001 C CNN
 F 3 "~" H 5450 3850 50  0001 C CNN
 	1    5450 3850
@@
 F 0 "D5" H 5993 4667 50  0000 C CNN
 F 1 "LED YELLOW" H 5993 4576 50  0000 C CNN
-F 2 "" H 6000 4450 50  0001 C CNN
+F 2 "LED_THT:LED_D5.0mm" H 6000 4450 50  0001 C CNN
 F 3 "~" H 6000 4450 50  0001 C CNN
 	1    6000 4450
@@
 F 0 "R2" V 7193 3900 50  0000 C CNN
 F 1 "330" V 7284 3900 50  0000 C CNN
-F 2 "" V 7330 3900 50  0001 C CNN
+F 2 "Resistor_THT:R_Axial_DIN0207_L6.3mm_D2.5mm_P7.62mm_Horizontal" V 7330 3900 50  0001 C CNN
 F 3 "~" H 7400 3900 50  0001 C CNN
 	1    7400 3900
@@
 F 0 "J1" H 2907 4217 50  0000 C CNN
 F 1 "Barrel_Jack_Switch" H 2907 4126 50  0000 C CNN
-F 2 "" H 2900 3860 50  0001 C CNN
+F 2 "Connector_BarrelJack:BarrelJack_CUI_PJ-102AH_Horizontal" H 2900 3860 50  0001 C CNN
 F 3 "~" H 2900 3860 50  0001 C CNN
 	1    2850 3900
@@
 F 0 "C1" H 4265 3896 50  0000 L CNN
 F 1 "470uF" H 4265 3805 50  0000 L CNN
-F 2 "" H 4150 3850 50  0001 C CNN
+F 2 "Capacitor_THT:CP_Radial_D10.0mm_P5.00mm" H 4150 3850 50  0001 C CNN
 F 3 "~" H 4150 3850 50  0001 C CNN
 	1    4150 3850
@@
 F 0 "D6" H 7393 4617 50  0000 C CNN
 F 1 "LED RED" H 7393 4526 50  0000 C CNN
-F 2 "" H 7400 4400 50  0001 C CNN
+F 2 "LED_THT:LED_D5.0mm" H 7400 4400 50  0001 C CNN
 F 3 "~" H 7400 4400 50  0001 C CNN
 	1    7400 4400
@@
 F 0 "R1" V 5793 3900 50  0000 C CNN
 F 1 "330" V 5884 3900 50  0000 C CNN
-F 2 "" V 5930 3900 50  0001 C CNN
+F 2 "Resistor_THT:R_Axial_DIN0207_L6.3mm_D2.5mm_P7.62mm_Horizontal" V 5930 3900 50  0001 C CNN
 F 3 "~" H 6000 3900 50  0001 C CNN
 	1    6000 3900
@@
 F 0 "SW1" H 6600 4285 50  0000 C CNN
 F 1 "SW_DPDT_x2" H 6600 4194 50  0000 C CNN
-F 2 "" H 6600 4000 50  0001 C CNN
+F 2 "digikey-footprints:Switch_Slide_11.6x4mm_EG1218" H 6600 4000 50  0001 C CNN
 F 3 "~" H 6600 4000 50  0001 C CNN
 	1    6600 4000
@@
 F 0 "J2" H 8250 4017 50  0000 C CNN
 F 1 "Conn_02x02_Odd_Even" H 8250 3926 50  0000 C CNN
-F 2 "" H 8200 3800 50  0001 C CNN
+F 2 "Connector_PinHeader_2.54mm:PinHeader_2x02_P2.54mm_Vertical" H 8200 3800 50  0001 C CNN
 F 3 "~" H 8200 3800 50  0001 C CNN
 	1    8200 3800
@@
 F 0 "J3" H 8250 4517 50  0000 C CNN
 F 1 "Conn_02x02_Odd_Even" H 8250 4426 50  0000 C CNN
-F 2 "" H 8200 4300 50  0001 C CNN
+F 2 "Connector_PinHeader_2.54mm:PinHeader_2x02_P2.54mm_Vertical" H 8200 4300 50  0001 C CNN
 F 3 "~" H 8200 4300 50  0001 C CNN
 	1    8200 4300

Commit message: Schematic ok
Parts:
- renumbered D6 to D5, D5 to D6
Connections:
- net Vin: now reaches U1.1 (VI)
- net Vin: now also C1.1, D1.1 (K), D3.1 (K)
- net GND: now reaches U1.2 (GND)
- net GND: now also C1.2, C2.2, D2.2 (A), D4.2 (A), D5.1 (K), D6.1 (K), J2.3 (Pin_3), J2.4 (Pin_4), J3.3 (Pin_3), J3.4 (Pin_4)
- net Vout1: now reaches U1.3 (VO)
- net Vout1: now also C2.1, R1.2, SW1.2 (B)
- net at D4.1 (K): now also D3.2 (A), J1.2
- net at D6.2 (A): now also R2.2
- net Vout2: now reaches R2.1
- net Vout2: now also J2.1 (Pin_1), J2.2 (Pin_2), J3.1 (Pin_1), J3.2 (Pin_2), SW1.1 (A)
- net at J1.1: now also D1.2 (A), D2.1 (K)
- net at D5.2 (A): now also R1.1
- no-connect marks 0 -> 2
Other:
- note added: "N1 - Power Input"
- note added: "N2 - Bridge Rectifier"
- note added: "N3 - Voltaje Regulator"
- note added: "N4 - \nPower \nIndicator"
- note added: "N5 - \nON/OFF\nSwitch"
- note added: "N6 -\nOutput\nPower\nIndicator"
- note added: "N7 - Power Output"
- moved on the sheet: C1, C2, D1, D2, D3, D4, D5, D6, J1, J2, J3, R1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

Commit message: Final PCB
Parts:
- D5, D6: footprint LED_THT:LED_D5.0mm -> LED_SMD:LED_0805_2012Metric
Changed lines of the file:
@@
 F 0 "D6" H 7600 3850 50  0000 C CNN
 F 1 "LED YELLOW" H 7593 4076 50  0000 C CNN
-F 2 "LED_THT:LED_D5.0mm" H 7600 3950 50  0001 C CNN
+F 2 "LED_SMD:LED_0805_2012Metric" H 7600 3950 50  0001 C CNN
 F 3 "~" H 7600 3950 50  0001 C CNN
 	1    7600 3950
@@
 F 0 "D5" H 6650 3850 50  0000 C CNN
 F 1 "LED RED" H 6643 4076 50  0000 C CNN
-F 2 "LED_THT:LED_D5.0mm" H 6650 3950 50  0001 C CNN
+F 2 "LED_SMD:LED_0805_2012Metric" H 6650 3950 50  0001 C CNN
 F 3 "~" H 6650 3950 50  0001 C CNN
 	1    6650 3950
