File: Raspberry Pi HAT/Raspberry Pi HAT.kicad_pcb (KiCad board)
At the start: 2 copper layers, 27.4 x 19.8 mm, 9 parts, among them J1 Raspberry_Pi_2_3, SW1 SW_DPST, U1 DHT22

Commit message: Wired
Parts:
- J1: footprint Connector_PinHeader_2.54mm:PinHeader_2x08_P2.54mm_Vertical -> Connector_PinSocket_2.54mm:PinSocket_2x08_P2.54mm_Vertical
- moved J1 2.54 mm to (112.3, 94.5)
Routing:
- net GND: track 0.00 -> 73.6 mm, vias 0 -> 3
- net VCC: track 0.00 -> 38.4 mm
- net Net-(J1-Pad7): track 0.00 -> 34.2 mm, vias 0 -> 1
- net /button_input: track 0.00 -> 21.2 mm, vias 0 -> 1
- net Net-(J1-Pad11): track 0.00 -> 20.7 mm
- net Net-(D1-Pad2): track 0.00 -> 2.57 mm
- added copper zone on B.Cu, net GND
- added copper zone on F.Cu, net GND

Commit message: finished
Parts:
- added REF**: OSHW-Logo2_7.3x6mm_SilkScreen, Symbol:OSHW-Logo2_7.3x6mm_SilkScreen, B.Cu at (124.2, 101.3)
- J1: footprint Connector_PinSocket_2.54mm:PinSocket_2x08_P2.54mm_Vertical -> Connector_PinHeader_2.54mm:PinHeader_2x08_P2.54mm_Vertical
- R1: value 330 -> 10k
- moved J1 2.54 mm to (112.4, 97.0)
Routing:
- net GND: track 73.6 -> 36.3 mm, vias 3 -> 1
- net VCC: track 38.4 -> 33.4 mm
- net Net-(J1-Pad7): track 34.2 -> 38.5 mm
- net /button_input: track 21.2 -> 25.1 mm, vias 1 -> 2
- net Net-(D2-Pad2): track 0.00 -> 2.95 mm
- net Net-(J1-Pad11): track 20.7 -> 18.0 mm
Other:
- board text added: "10K"
- board text added: "10k"
- board text added: "330"
- board text added: "Author: Diego Gonzales"
- board text added: "Button: GPIO14 LED: GPIO4"
- board text added: "GPIO14/Pin8"
- board text added: "PWR"
- board text added: "Raspberry Pi HAT v1.0"
