File: Raspberry Pi HAT/Raspberry Pi HAT.kicad_pcb (KiCad board)
At the start: 2 copper layers, 27.4 x 19.8 mm, 10 parts, among them J1 Raspberry_Pi_2_3, SW1 SW_DPST, U1 DHT22

Commit message: extra files
Parts:
- removed REF**: OSHW-Logo2_7.3x6mm_SilkScreen, Symbol:OSHW-Logo2_7.3x6mm_SilkScreen
- added G***: LOGO, logos:Catcuber_4.9x4.9mm, B.Cu at (124.2, 102.1)
