File: Raspberry Pi HAT/Raspberry Pi HAT.sch (KiCad schematic (older format))
At the start: 7 parts, among them J1 Raspberry_Pi_2_3, SW1 SW_DPST, U1 DHT22

Commit message: Schema finished
Parts:
- added D2: LED RED, LED_SMD:LED_0805_2012Metric, symbol Device:LED
- added R4: 330, Resistor_SMD:R_0805_2012Metric, symbol Device:R
Connections:
- net VCC: now reaches J1.1 (3V3)
- net VCC: now also R2.2, SW1.1, SW1.3, U1.1 (VCC), R4.1
- net at J1.11 (GPIO17): now also R2.1, U1.2 (IO)
- net GND: now reaches J1.6 (GND)
- net GND: now also D1.1 (K), J1.9 (GND), R1.2, U1.4 (GND), D2.1 (K)
- net at J1.7 (GCLK0/GPIO4): now also R3.1
- net button_input: now reaches J1.8 (GPIO14/TXD)
- net button_input: now also R1.1, SW1.2, SW1.4
- net at R3.2: now also D1.2 (A)
- new net: D2.2 (A), R4.2
- no-connect marks 0 -> 34
Other:
- note added: "N1 - Button"
- note added: "N2 - Sensor DTH22"
- note added: "N3 - Raspberry Pi"
- note added: "N4 - Indicator LED"
- note added: "N5 - Power LED"
- moved on the sheet: D1, J1, R1, R2, R3, SW1, U1

Commit message: finished
Parts:
- J1: footprint Connector_PinSocket_2.54mm:PinSocket_2x08_P2.54mm_Vertical -> Connector_PinHeader_2.54mm:PinHeader_2x08_P2.54mm_Vertical
- R1: value 330 -> 10k
Changed lines of the file:
@@
 F 0 "J1" H 7050 4900 50  0000 C CNN
 F 1 "Raspberry_Pi_2_3" H 7050 4800 50  0000 C CNN
-F 2 "Connector_PinSocket_2.54mm:PinSocket_2x08_P2.54mm_Vertical" H 6450 3500 50  0001 C CNN
+F 2 "Connector_PinHeader_2.54mm:PinHeader_2x08_P2.54mm_Vertical" H 6450 3500 50  0001 C CNN
 F 3 "https://www.raspberrypi.org/documentation/hardware/raspberrypi/schematics/rpi_SCH_3bplus_1p0_reduced.pdf" H 6450 3500 50  0001 C CNN
 	1    6450 3500
@@
 P 3550 3400
 F 0 "R1" H 3620 3446 50  0000 L CNN
-F 1 "330" H 3620 3355 50  0000 L CNN
+F 1 "10k" H 3620 3355 50  0000 L CNN
 F 2 "Resistor_SMD:R_0805_2012Metric" V 3480 3400 50  0001 C CNN
 F 3 "~" H 3550 3400 50  0001 C CNN
