File: Arduino Clone/_autosave-Arduino Clone.sch (KiCad schematic (older format))
At the start: 6 parts

Commit message: xd
Parts:
- added U?: ATmega328P-AU, Package_QFP:TQFP-32_7x7mm_P0.8mm, symbol MCU_Microchip_ATmega:ATmega328P-AU
Connections:
- new net: U?.21 (GND), U?.3 (GND), U?.5 (GND)
- new net: U?.4 (VCC), U?.6 (VCC)
Other:
- moved on the sheet: BT?, C?, D?, U?
Changed lines of the file:
@@
 L Device:Battery BT?
 U 1 1 5FCEA658
-P 1950 3200
-F 0 "BT?" H 2058 3246 50  0000 L CNN
-F 1 "Battery" H 2058 3155 50  0000 L CNN
-F 2 "" V 1950 3260 50  0001 C CNN
-F 3 "~" V 1950 3260 50  0001 C CNN
-	1    1950 3200
+P 3900 2200
+F 0 "BT?" H 4008 2246 50  0000 L CNN
+F 1 "Battery" H 4008 2155 50  0000 L CNN
+F 2 "" V 3900 2260 50  0001 C CNN
+F 3 "~" V 3900 2260 50  0001 C CNN
+	1    3900 2200
 	1    0    0    -1
 $EndComp
@@
 L Device:C C?
 U 1 1 5FCEB637
-P 2650 3000
-F 0 "C?" H 2765 3046 50  0000 L CNN
-F 1 "C" H 2765 2955 50  0000 L CNN
-F 2 "" H 2688 2850 50  0001 C CNN
-F 3 "~" H 2650 3000 50  0001 C CNN
-	1    2650 3000
+P 4600 2000
+F 0 "C?" H 4715 2046 50  0000 L CNN
+F 1 "C" H 4715 1955 50  0000 L CNN
+F 2 "" H 4638 1850 50  0001 C CNN
+F 3 "~" H 4600 2000 50  0001 C CNN
+	1    4600 2000
 	1    0    0    -1
 $EndComp
@@
 L Device:C C?
 U 1 1 5FCEBC26
-P 3000 3000
-F 0 "C?" H 3115 3046 50  0000 L CNN
-F 1 "C" H 3115 2955 50  0000 L CNN
-F 2 "" H 3038 2850 50  0001 C CNN
-F 3 "~" H 3000 3000 50  0001 C CNN
-	1    3000 3000
+P 4950 2000
+F 0 "C?" H 5065 2046 50  0000 L CNN
+F 1 "C" H 5065 1955 50  0000 L CNN
+F 2 "" H 4988 1850 50  0001 C CNN
+F 3 "~" H 4950 2000 50  0001 C CNN
+	1    4950 2000
 	1    0    0    -1
 $EndComp
@@
 L Device:CP C?
 U 1 1 5FCEBFBC
-P 2650 3450
-F 0 "C?" H 2768 3496 50  0000 L CNN
-F 1 "CP" H 2768 3405 50  0000 L CNN
-F 2 "" H 2688 3300 50  0001 C CNN
-F 3 "~" H 2650 3450 50  0001 C CNN
-	1    2650 3450
+P 4600 2450
+F 0 "C?" H 4718 2496 50  0000 L CNN
+F 1 "CP" H 4718 2405 50  0000 L CNN
+F 2 "" H 4638 2300 50  0001 C CNN
+F 3 "~" H 4600 2450 50  0001 C CNN
+	1    4600 2450
 	1    0    0    -1
 $EndComp
@@
 L Device:LED D?
 U 1 1 5FCEC229
-P 3500 3150
-F 0 "D?" H 3493 3367 50  0000 C CNN
-F 1 "LED" H 3493 3276 50  0000 C CNN
-F 2 "" H 3500 3150 50  0001 C CNN
-F 3 "~" H 3500 3150 50  0001 C CNN
-	1    3500 3150
+P 5450 2150
+F 0 "D?" H 5443 2367 50  0000 C CNN
+F 1 "LED" H 5443 2276 50  0000 C CNN
+F 2 "" H 5450 2150 50  0001 C CNN
+F 3 "~" H 5450 2150 50  0001 C CNN
+	1    5450 2150
 	1    0    0    -1
 $EndComp
@@
 L Memory_EEPROM:24LC1025 U?
 U 1 1 5FCED1F5
-P 4300 3050
-F 0 "U?" H 4300 3531 50  0000 C CNN
-F 1 "24LC1025" H 4300 3440 50  0000 C CNN
-F 2 "" H 4300 3050 50  0001 C CNN
-F 3 "http://ww1.microchip.com/downloads/en/DeviceDoc/21941B.pdf" H 4300 3050 50  0001 C CNN
-	1    4300 3050
+P 6250 2050
+F 0 "U?" H 6250 2531 50  0000 C CNN
+F 1 "24LC1025" H 6250 2440 50  0000 C CNN
+F 2 "" H 6250 2050 50  0001 C CNN
+F 3 "http://ww1.microchip.com/downloads/en/DeviceDoc/21941B.pdf" H 6250 2050 50  0001 C CNN
+	1    6250 2050
 	1    0    0    -1
 $EndComp
 $Sheet
-S 5250 2800 2250 1500
+S 6800 2800 2250 1500
 U 5FCEF225
 F0 "Connectors" 50
 F1 "Connectors.sch" 50
 $EndSheet
+$Comp
+L MCU_Microchip_ATmega:ATmega328P-AU U?
+U 1 1 5FCF2F91
+P 4300 4500
+F 0 "U?" H 4300 2911 50  0000 C CNN
+F 1 "ATmega328P-AU" H 4300 2820 50  0000 C CNN
+F 2 "Package_QFP:TQFP-32_7x7mm_P0.8mm" H 4300 4500 50  0001 C CIN
+F 3 "http://ww1.microchip.com/downloads/en/DeviceDoc/ATmega328_P%20AVR%20MCU%20with%20picoPower%20Technology%20Data%20Sheet%2040001984A.pdf" H 4300 4500 50  0001 C CNN
+	1    4300 4500
+	1    0    0    -1
+$EndComp
 $EndSCHEMATC
