File: Arduino Clone/Arduino Clone.sch (KiCad schematic (older format))
At the start: 6 parts

Commit message: 30%
Parts:
- added R1, R2: R, Resistor_SMD:R_0805_2012Metric, symbol Device:R
- added U2: 24LC1025, Package_SO:SOIJ-8_5.3x5.3mm_P1.27mm, symbol Memory_EEPROM:24LC1025
- added U3: DS1337_my, Package_SO:SO-8_5.3x6.2mm_P1.27mm, symbol my~libraries:DS1337_my
- added U4: ATmega328P-AU, Package_QFP:TQFP-32_7x7mm_P0.8mm, symbol MCU_Microchip_ATmega:ATmega328P-AU
- added Y1: Crystal, Crystal:Crystal_SMD_MicroCrystal_CC7V-T1A-2Pin_3.2x1.5mm, symbol Device:Crystal
- added Y2: Crystal, Crystal:Crystal_SMD_5032-2Pin_5.0x3.2mm_HandSoldering, symbol Device:Crystal
- BT1: renamed from BT?; footprint (none) -> Connector_JST:JST_EH_B2B-EH-A_1x02_P2.50mm_Vertical
- C1, C2, C3: renamed from C?; footprint (none) -> Capacitor_SMD:C_0805_2012Metric
- D1: renamed from D?; footprint (none) -> LED_SMD:LED_0805_2012Metric
- U1: renamed from U?; footprint (none) -> Package_SO:SOIJ-8_5.3x5.3mm_P1.27mm
Other:
- moved on the sheet: BT1, C1, C2, C3, D1, U1
Changed lines of the file:
@@
 $EndBitmap
 $Comp
-L Device:Battery BT?
+L Device:Battery BT1
 U 1 1 5FCEA658
-P 1950 3200
-F 0 "BT?" H 2058 3246 50  0000 L CNN
-F 1 "Battery" H 2058 3155 50  0000 L CNN
-F 2 "" V 1950 3260 50  0001 C CNN
-F 3 "~" V 1950 3260 50  0001 C CNN
-	1    1950 3200
+P 9050 2200
+F 0 "BT1" H 9158 2246 50  0000 L CNN
+F 1 "Battery" H 9158 2155 50  0000 L CNN
+F 2 "Connector_JST:JST_EH_B2B-EH-A_1x02_P2.50mm_Vertical" V 9050 2260 50  0001 C CNN
+F 3 "~" V 9050 2260 50  0001 C CNN
+	1    9050 2200
 	1    0    0    -1
 $EndComp
 $Comp
-L Device:C C?
+L Device:C C2
 U 1 1 5FCEB637
-P 2650 3000
-F 0 "C?" H 2765 3046 50  0000 L CNN
-F 1 "C" H 2765 2955 50  0000 L CNN
-F 2 "" H 2688 2850 50  0001 C CNN
-F 3 "~" H 2650 3000 50  0001 C CNN
-	1    2650 3000
+P 6250 3200
+F 0 "C2" H 6365 3246 50  0000 L CNN
+F 1 "C" H 6365 3155 50  0000 L CNN
+F 2 "Capacitor_SMD:C_0805_2012Metric" H 6288 3050 50  0001 C CNN
+F 3 "~" H 6250 3200 50  0001 C CNN
+	1    6250 3200
 	1    0    0    -1
 $EndComp
 $Comp
-L Device:C C?
+L Device:C C1
 U 1 1 5FCEBC26
-P 3000 3000
-F 0 "C?" H 3115 3046 50  0000 L CNN
-F 1 "C" H 3115 2955 50  0000 L CNN
-F 2 "" H 3038 2850 50  0001 C CNN
-F 3 "~" H 3000 3000 50  0001 C CNN
-	1    3000 3000
+P 6250 2700
+F 0 "C1" H 6365 2746 50  0000 L CNN
+F 1 "C" H 6365 2655 50  0000 L CNN
+F 2 "Capacitor_SMD:C_0805_2012Metric" H 6288 2550 50  0001 C CNN
+F 3 "~" H 6250 2700 50  0001 C CNN
+	1    6250 2700
 	1    0    0    -1
 $EndComp
 $Comp
-L Device:CP C?
+L Device:CP C3
 U 1 1 5FCEBFBC
-P 2650 3450
-F 0 "C?" H 2768 3496 50  0000 L CNN
-F 1 "CP" H 2768 3405 50  0000 L CNN
-F 2 "" H 2688 3300 50  0001 C CNN
-F 3 "~" H 2650 3450 50  0001 C CNN
-	1    2650 3450
+P 9750 2450
+F 0 "C3" H 9868 2496 50  0000 L CNN
+F 1 "CP" H 9868 2405 50  0000 L CNN
+F 2 "Capacitor_SMD:C_0805_2012Metric" H 9788 2300 50  0001 C CNN
+F 3 "~" H 9750 2450 50  0001 C CNN
+	1    9750 2450
 	1    0    0    -1
 $EndComp
 $Comp
-L Device:LED D?
+L Device:LED D1
 U 1 1 5FCEC229
-P 3500 3150
-F 0 "D?" H 3493 3367 50  0000 C CNN
-F 1 "LED" H 3493 3276 50  0000 C CNN
-F 2 "" H 3500 3150 50  0001 C CNN
-F 3 "~" H 3500 3150 50  0001 C CNN
-	1    3500 3150
+P 6350 3800
+F 0 "D1" H 6343 4017 50  0000 C CNN
+F 1 "LED" H 6343 3926 50  0000 C CNN
+F 2 "LED_SMD:LED_0805_2012Metric" H 6350 3800 50  0001 C CNN
+F 3 "~" H 6350 3800 50  0001 C CNN
+	1    6350 3800
 	1    0    0    -1
 $EndComp
 $Comp
-L Memory_EEPROM:24LC1025 U?
+L Memory_EEPROM:24LC1025 U1
 U 1 1 5FCED1F5
-P 4300 3050
-F 0 "U?" H 4300 3531 50  0000 C CNN
-F 1 "24LC1025" H 4300 3440 50  0000 C CNN
-F 2 "" H 4300 3050 50  0001 C CNN
-F 3 "http://ww1.microchip.com/downloads/en/DeviceDoc/21941B.pdf" H 4300 3050 50  0001 C CNN
-	1    4300 3050
+P 2050 5350
+F 0 "U1" H 2050 5831 50  0000 C CNN
+F 1 "24LC1025" H 2050 5740 50  0000 C CNN
+F 2 "Package_SO:SOIJ-8_5.3x5.3mm_P1.27mm" H 2050 5350 50  0001 C CNN
+F 3 "http://ww1.microchip.com/downloads/en/DeviceDoc/21941B.pdf" H 2050 5350 50  0001 C CNN
+	1    2050 5350
 	1    0    0    -1
 $EndComp
 $Sheet
-S 5250 2800 2250 1500
+S 8300 4650 2250 1500
 U 5FCEF225
 F0 "Connectors" 50
 F1 "Connectors.sch" 50
 $EndSheet
+$Comp
+L MCU_Microchip_ATmega:ATmega328P-AU U4
+U 1 1 5FCF2F91
+P 5100 3600
+F 0 "U4" H 5100 2011 50  0000 C CNN
+F 1 "ATmega328P-AU" H 5100 1920 50  0000 C CNN
+F 2 "Package_QFP:TQFP-32_7x7mm_P0.8mm" H 5100 3600 50  0001 C CIN
+F 3 "http://ww1.microchip.com/downloads/en/DeviceDoc/ATmega328_P%20AVR%20MCU%20with%20picoPower%20Technology%20Data%20Sheet%2040001984A.pdf" H 5100 3600 50  0001 C CNN
+	1    5100 3600
+	1    0    0    -1
+$EndComp
+$Comp
+L my~libraries:DS1337_my U3
+U 1 1 5FCF679E
+P 2300 3650
+F 0 "U3" H 2300 4231 50  0000 C CNN
+F 1 "DS1337_my" H 2300 4140 50  0000 C CNN
+F 2 "Package_SO:SO-8_5.3x6.2mm_P1.27mm" H 2300 3650 50  0001 C CNN
+F 3 "" H 2300 3650 50  0001 C CNN
+	1    2300 3650
+	1    0    0    -1
+$EndComp
+$Comp
+L Device:Crystal Y2
+U 1 1 5FCF85D4
+P 6800 2950
+F 0 "Y2" H 6800 3218 50  0000 C CNN
+F 1 "Crystal" H 6800 3127 50  0000 C CNN
+F 2 "Crystal:Crystal_SMD_5032-2Pin_5.0x3.2mm_HandSoldering" H 6800 2950 50  0001 C CNN
+F 3 "~" H 6800 2950 50  0001 C CNN
+	1    6800 2950
+	0    -1   -1   0
+$EndComp
+$Comp
+L Device:Crystal Y1
+U 1 1 5FCF886F
+P 1550 3450
+F 0 "Y1" H 1550 3718 50  0000 C CNN
+F 1 "Crystal" H 1550 3627 50  0000 C CNN
+F 2 "Crystal:Crystal_SMD_MicroCrystal_CC7V-T1A-2Pin_3.2x1.5mm" H 1550 3450 50  0001 C CNN
+F 3 "~" H 1550 3450 50  0001 C CNN
+	1    1550 3450
+	1    0    0    -1
+$EndComp
+$Comp
+L Memory_EEPROM:24LC1025 U2
+U 1 1 5FCF9FF3
+P 2050 6200
+F 0 "U2" H 2050 6681 50  0000 C CNN
+F 1 "24LC1025" H 2050 6590 50  0000 C CNN
+F 2 "Package_SO:SOIJ-8_5.3x5.3mm_P1.27mm" H 2050 6200 50  0001 C CNN
+F 3 "http://ww1.microchip.com/downloads/en/DeviceDoc/21941B.pdf" H 2050 6200 50  0001 C CNN
+	1    2050 6200
+	1    0    0    -1
+$EndComp
+$Comp
+L Device:R R2
+U 1 1 5FD01D54
+P 8400 2350
+F 0 "R2" H 8470 2396 50  0000 L CNN
+F 1 "R" H 8470 2305 50  0000 L CNN
+F 2 "Resistor_SMD:R_0805_2012Metric" V 8330 2350 50  0001 C CNN
+F 3 "~" H 8400 2350 50  0001 C CNN
+	1    8400 2350
+	1    0    0    -1
+$EndComp
+$Comp
+L Device:R R1
+U 1 1 5FD01F7E
+P 6700 3900
+F 0 "R1" H 6770 3946 50  0000 L CNN
+F 1 "R" H 6770 3855 50  0000 L CNN
+F 2 "Resistor_SMD:R_0805_2012Metric" V 6630 3900 50  0001 C CNN
+F 3 "~" H 6700 3900 50  0001 C CNN
+	1    6700 3900
+	1    0    0    -1
+$EndComp
 $EndSCHEMATC

Commit message: hierarchical label
Parts:
- BT1: value Battery -> Battery 3v
- C1, C2: value C -> 22pF
- C3: value CP -> 10uF
- R1: value R -> 330Ohm
- R2: value R -> 10kOhm
- U3: value DS1337_my -> DS1337
- Y1: value Crystal -> Crystal 32MHz
- Y2: value Crystal -> Crystal 16MHz
Connections:
- net labels added: D2, D3, D4, D5, D6, D7, D8, GND, GNDPWR, MISO, MOSI, RESET, Rx, SCK, SDA, Tx, Vcc
- wire segments 0 -> 24
Other:
- moved on the sheet: C1, C2, D1, R1, Y2
Changed lines of the file:
@@
 P 9050 2200
 F 0 "BT1" H 9158 2246 50  0000 L CNN
-F 1 "Battery" H 9158 2155 50  0000 L CNN
+F 1 "Battery 3v" H 9158 2155 50  0000 L CNN
 F 2 "Connector_JST:JST_EH_B2B-EH-A_1x02_P2.50mm_Vertical" V 9050 2260 50  0001 C CNN
 F 3 "~" V 9050 2260 50  0001 C CNN
@@
 L Device:C C2
 U 1 1 5FCEB637
-P 6250 3200
-F 0 "C2" H 6365 3246 50  0000 L CNN
-F 1 "C" H 6365 3155 50  0000 L CNN
-F 2 "Capacitor_SMD:C_0805_2012Metric" H 6288 3050 50  0001 C CNN
-F 3 "~" H 6250 3200 50  0001 C CNN
-	1    6250 3200
+P 6300 3200
+F 0 "C2" H 6415 3246 50  0000 L CNN
+F 1 "22pF" H 6415 3155 50  0000 L CNN
+F 2 "Capacitor_SMD:C_0805_2012Metric" H 6338 3050 50  0001 C CNN
+F 3 "~" H 6300 3200 50  0001 C CNN
+	1    6300 3200
 	1    0    0    -1
 $EndComp
@@
 L Device:C C1
 U 1 1 5FCEBC26
-P 6250 2700
-F 0 "C1" H 6365 2746 50  0000 L CNN
-F 1 "C" H 6365 2655 50  0000 L CNN
-F 2 "Capacitor_SMD:C_0805_2012Metric" H 6288 2550 50  0001 C CNN
-F 3 "~" H 6250 2700 50  0001 C CNN
-	1    6250 2700
+P 6300 2700
+F 0 "C1" H 6415 2746 50  0000 L CNN
+F 1 "22pF" H 6415 2655 50  0000 L CNN
+F 2 "Capacitor_SMD:C_0805_2012Metric" H 6338 2550 50  0001 C CNN
+F 3 "~" H 6300 2700 50  0001 C CNN
+	1    6300 2700
 	1    0    0    -1
 $EndComp
@@
 P 9750 2450
 F 0 "C3" H 9868 2496 50  0000 L CNN
-F 1 "CP" H 9868 2405 50  0000 L CNN
+F 1 "10uF" H 9868 2405 50  0000 L CNN
 F 2 "Capacitor_SMD:C_0805_2012Metric" H 9788 2300 50  0001 C CNN
 F 3 "~" H 9750 2450 50  0001 C CNN
@@
 L Device:LED D1
 U 1 1 5FCEC229
-P 6350 3800
-F 0 "D1" H 6343 4017 50  0000 C CNN
-F 1 "LED" H 6343 3926 50  0000 C CNN
-F 2 "LED_SMD:LED_0805_2012Metric" H 6350 3800 50  0001 C CNN
-F 3 "~" H 6350 3800 50  0001 C CNN
-	1    6350 3800
+P 6400 3800
+F 0 "D1" H 6393 4017 50  0000 C CNN
+F 1 "LED" H 6393 3926 50  0000 C CNN
+F 2 "LED_SMD:LED_0805_2012Metric" H 6400 3800 50  0001 C CNN
+F 3 "~" H 6400 3800 50  0001 C CNN
+	1    6400 3800
 	1    0    0    -1
 $EndComp
@@
 	1    0    0    -1
 $EndComp
-$Sheet
-S 8300 4650 2250 1500
-U 5FCEF225
-F0 "Connectors" 50
-F1 "Connectors.sch" 50
-$EndSheet
 $Comp
 L MCU_Microchip_ATmega:ATmega328P-AU U4
 U 1 1 5FCF2F91
 P 5100 3600
-F 0 "U4" H 5100 2011 50  0000 C CNN
-F 1 "ATmega328P-AU" H 5100 1920 50  0000 C CNN
+F 0 "U4" H 5100 1850 50  0000 C CNN
+F 1 "ATmega328P-AU" H 5100 1750 50  0000 C CNN
 F 2 "Package_QFP:TQFP-32_7x7mm_P0.8mm" H 5100 3600 50  0001 C CIN
 F 3 "http://ww1.microchip.com/downloads/en/DeviceDoc/ATmega328_P%20AVR%20MCU%20with%20picoPower%20Technology%20Data%20Sheet%2040001984A.pdf" H 5100 3600 50  0001 C CNN
@@
 P 2300 3650
 F 0 "U3" H 2300 4231 50  0000 C CNN
-F 1 "DS1337_my" H 2300 4140 50  0000 C CNN
+F 1 "DS1337" H 2300 4140 50  0000 C CNN
 F 2 "Package_SO:SO-8_5.3x6.2mm_P1.27mm" H 2300 3650 50  0001 C CNN
 F 3 "" H 2300 3650 50  0001 C CNN
@@
 L Device:Crystal Y2
 U 1 1 5FCF85D4
-P 6800 2950
-F 0 "Y2" H 6800 3218 50  0000 C CNN
-F 1 "Crystal" H 6800 3127 50  0000 C CNN
-F 2 "Crystal:Crystal_SMD_5032-2Pin_5.0x3.2mm_HandSoldering" H 6800 2950 50  0001 C CNN
-F 3 "~" H 6800 2950 50  0001 C CNN
-	1    6800 2950
+P 6850 2950
+F 0 "Y2" H 6850 3218 50  0000 C CNN
+F 1 "Crystal 16MHz" H 6850 3127 50  0000 C CNN
+F 2 "Crystal:Crystal_SMD_5032-2Pin_5.0x3.2mm_HandSoldering" H 6850 2950 50  0001 C CNN
+F 3 "~" H 6850 2950 50  0001 C CNN
+	1    6850 2950
 	0    -1   -1   0
 $EndComp
@@
 P 1550 3450
 F 0 "Y1" H 1550 3718 50  0000 C CNN
-F 1 "Crystal" H 1550 3627 50  0000 C CNN
+F 1 "Crystal 32MHz" H 1550 3627 50  0000 C CNN
 F 2 "Crystal:Crystal_SMD_MicroCrystal_CC7V-T1A-2Pin_3.2x1.5mm" H 1550 3450 50  0001 C CNN
 F 3 "~" H 1550 3450 50  0001 C CNN
@@
 P 8400 2350
 F 0 "R2" H 8470 2396 50  0000 L CNN
-F 1 "R" H 8470 2305 50  0000 L CNN
+F 1 "10kOhm" H 8470 2305 50  0000 L CNN
 F 2 "Resistor_SMD:R_0805_2012Metric" V 8330 2350 50  0001 C CNN
 F 3 "~" H 8400 2350 50  0001 C CNN
@@
 L Device:R R1
 U 1 1 5FD01F7E
-P 6700 3900
-F 0 "R1" H 6770 3946 50  0000 L CNN
-F 1 "R" H 6770 3855 50  0000 L CNN
-F 2 "Resistor_SMD:R_0805_2012Metric" V 6630 3900 50  0001 C CNN
-F 3 "~" H 6700 3900 50  0001 C CNN
-	1    6700 3900
-	1    0    0    -1
-$EndComp
+P 6750 3900
+F 0 "R1" H 6820 3946 50  0000 L CNN
+F 1 "330Ohm" H 6820 3855 50  0000 L CNN
+F 2 "Resistor_SMD:R_0805_2012Metric" V 6680 3900 50  0001 C CNN
+F 3 "~" H 6750 3900 50  0001 C CNN
+	1    6750 3900
+	1    0    0    -1
+$EndComp
+Text Label 7350 4700 2    50   ~ 0
+MISO
+Wire Wire Line
+	7350 4700 7550 4700
+$Sheet
+S 7550 4600 2250 1500
+U 5FCEF225
+F0 "Connectors" 50
+F1 "Connectors.sch" 50
+F2 "MISO" O L 7550 4700 50
+F3 "SCK" B L 7550 4850 50
+F4 "RESET" O L 7550 5150 50
+F5 "Vcc" I L 7550 5750 50
+F6 "MOSI" I L 7550 5000 50
+F7 "GND" I L 7550 5900 50
+F8 "Rx" I L 7550 5300 50
+F9 "Tx" O L 7550 5450 50
+F10 "SDA" B R 9800 4700 50
+F11 "D2" B R 9800 5000 50
+F12 "D3" B R 9800 5150 50
+F13 "D4" B R 9800 5300 50
+F14 "D5" B R 9800 5450 50
+F15 "D6" B R 9800 5600 50
+F16 "D7" B R 9800 5750 50
+F17 "D8" B R 9800 5900 50
+$EndSheet
+Text Label 5700 2800 0    50   ~ 0
+MISO
+Text Label 7350 4850 2    50   ~ 0
+SCK
+Text Label 7350 5150 2    50   ~ 0
+RESET
+Text Label 7350 5750 2    50   ~ 0
+Vcc
+Text Label 7350 5000 2    50   ~ 0
+MOSI
+Text Label 7350 5900 2    50   ~ 0
+GND
+Wire Wire Line
+	7350 4850 7550 4850
+Wire Wire Line
+	7350 5150 7550 5150
+Wire Wire Line
+	7350 5750 7550 5750
+Wire Wire Line
+	7350 5000 7550 5000
+Wire Wire Line
+	7350 5900 7400 5900
+Text Label 5700 2700 0    50   ~ 0
+MOSI
+Text Label 5700 2900 0    50   ~ 0
+SCK
+Text Label 5700 3900 0    50   ~ 0
+RESET
+Text Label 5100 1900 2    50   ~ 0
+Vcc
+Wire Wire Line
+	5100 2100 5100 1950
+Text Label 5000 5200 2    50   ~ 0
+GND
+$Comp
+L power:GNDPWR #PWR?
+U 1 1 5FDAD4AA
+P 7400 6050
+F 0 "#PWR?" H 7400 5850 50  0001 C CNN
+F 1 "GNDPWR" H 7404 5896 50  0000 C CNN
+F 2 "" H 7400 6000 50  0001 C CNN
+F 3 "" H 7400 6000 50  0001 C CNN
+	1    7400 6050
+	1    0    0    -1
+$EndComp
+Wire Wire Line
+	7400 6050 7400 5900
+Connection ~ 7400 5900
+Wire Wire Line
+	7400 5900 7550 5900
+Wire Wire Line
+	5200 2100 5200 1950
+Wire Wire Line
+	5200 1950 5100 1950
+Connection ~ 5100 1950
+Wire Wire Line
+	5100 1950 5100 1900
+Wire Wire Line
+	5000 5200 5100 5200
+Wire Wire Line
+	5100 5200 5100 5100
+Text Label 10050 4700 0    50   ~ 0
+SDA
+Text Label 10050 5000 0    50   ~ 0
+D2
+Text Label 10050 5150 0    50   ~ 0
+D3
+Text Label 10050 5300 0    50   ~ 0
+D4
+Text Label 10050 5450 0    50   ~ 0
+D5
+Text Label 10050 5600 0    50   ~ 0
+D6
+Text Label 10050 5750 0    50   ~ 0
+D7
+Text Label 10050 5900 0    50   ~ 0
+D8
+Text Label 7350 5300 2    50   ~ 0
+Rx
+Text Label 7350 5450 2    50   ~ 0
+Tx
+Wire Wire Line
+	7350 5300 7550 5300
+Wire Wire Line
+	7350 5450 7550 5450
+Wire Wire Line
+	10050 4700 9800 4700
+Wire Wire Line
+	10050 5000 9800 5000
+Wire Wire Line
+	9800 5150 10050 5150
+Wire Wire Line
+	10050 5300 9800 5300
+Wire Wire Line
+	10050 5450 9800 5450
+Wire Wire Line
+	9800 5600 10050 5600
+Wire Wire Line
+	10050 5750 9800 5750
+Wire Wire Line
+	9800 5900 10050 5900
+Text Label 5700 4400 0    50   ~ 0
+D3
+Text Label 5700 4500 0    50   ~ 0
+D4
+Text Label 5700 4600 0    50   ~ 0
+D5
+Text Label 5700 4700 0    50   ~ 0
+D6
+Text Label 5700 4800 0    50   ~ 0
+D7
+Text Label 5700 2400 0    50   ~ 0
+D8
+Text Label 5700 3700 0    50   ~ 0
+SDA
+Text Label 5700 4100 0    50   ~ 0
+Rx
+Text Label 5700 4200 0    50   ~ 0
+Tx
+Text Label 5700 4300 0    50   ~ 0
+D2
 $EndSCHEMATC

Commit message: finish ruting
Connections:
- net labels added: ADDS1, ADDS2, SCL
- wire segments 24 -> 79
- no-connect marks 0 -> 7
Other:
- moved on the sheet: BT1, C1, C2, C3, D1, R1, R2, U1, U2, U4, Y1, Y2

Commit message: labels
Other:
- note added: "N1 - Connectors"
- note added: "N2 - EEPROM"
- note added: "N3 - Atmega328p-AU with oscilator"
- note added: "N4 - Battery"
- note added: "N5 - Clock/Calendat"
- moved on the sheet: BT1, C1, C2, C3, D1, R1, R2, U1, U2, U4, Y1, Y2
