File: Led and Resistor/Led and Resistor.kicad_pcb (KiCad board)
At the start: 2 copper layers, 54.6 x 15.2 mm, 4 parts

Commit message: Breadboard Power Supply
Parts:
- removed the REF** at (151.1, 106.7)
- added J1: Conn_01x02_Male, TerminalBlock:TerminalBlock_bornier-2_P5.08mm, F.Cu at (151.1, 106.7)
Routing:
- net Net-(D1-Pad2): track 11.2 -> 31.0 mm
- net (no net): track 15.2 -> 0.00 mm
- net +5V: track 0.00 -> 14.0 mm
Other:
- net class PWR added: clearance 0.2, trace_width 0.4, via_dia 0.8, via_drill 0.4

Commit message: .
Parts:
- added G***: LOGO, logos:Catcuber_10.9x10.9mm, B.Cu at (154.8, 108.5)
